Commit message: switch to skid steer

File: my_robot/urdf/sad_robot.xacro (robot description, xacro)
@@ -1,5 +1,5 @@
 <?xml version='1.0'?>
-<robot name="my_robot" xmlns:xacro="http://www.ros.org/wiki/xacro">
-    <xacro:include filename="$(find my_robot)/urdf/my_robot.gazebo"/>
+<robot name="sad_robot" xmlns:xacro="http://www.ros.org/wiki/xacro">
+    <xacro:include filename="$(find my_robot)/urdf/sad_robot.gazebo"/>
     <link name="robot_footprint"/>
     <joint name="robot_footprint_joint" type="fixed">
@@ -11,9 +11,9 @@
         <pose> 0 0 0 0 0 0</pose>
         <inertial>
-            <mass value="8.0"/>
-            <origin xyz="0 0 0" rpy="0 0 0"/>
-            <inertia ixx="0.3"
-                     iyy="0.3"
-                     izz="0.1"
+            <mass value="15.0"/>
+            <origin xyz="0 0 0" rpy="0 0 0"/>
+            <inertia ixx="1.8"
+                     iyy="1.8"
+                     izz="1.3"
                      ixy="0.0" ixz="0.0" iyz="0.0"
                      />
@@ -40,9 +40,9 @@
         <pose> 0 0 0 0 0 0</pose>
         <inertial>
-            <mass value="0.2"/>
-            <origin xyz="0 0 0" rpy="0 0 0"/>
-            <inertia ixx="0.1"
-                     iyy="0.1"
-                     izz="0.1"
+            <mass value="0.6"/>
+            <origin xyz="0 0 0" rpy="0 0 0"/>
+            <inertia ixx="0.9"
+                     iyy="0.9"
+                     izz="0.6"
                      ixy="0.0" ixz="0.0" iyz="0.0"
                      />
@@ -365,5 +365,5 @@
         </collision>
         <inertial>
-            <mass value="1.0"/>
+            <mass value="2.0"/>
             <origin xyz="0 0 0" rpy="0 1.5707 1.5707"/>
             <inertia
@@ -389,5 +389,5 @@
         </collision>
         <inertial>
-            <mass value="1.0"/>
+            <mass value="2.0"/>
             <origin xyz="0 0 0" rpy="0 1.5707 1.5707"/>
             <inertia
@@ -405,59 +405,4 @@
         </visual>
     </link>
-    <!-- Strut dims are derived from the dims of the wheel they carry -->
-    <link name="front_left_strut">
-        <collision>
-            <origin xyz="0 0 0" rpy="0 0 0"/>
-            <geometry>
-                <box size='0.03 0.03 0.1'/>
-            </geometry>
-        </collision>
-        <inertial>
-            <mass value="0.2"/>
-            <origin xyz="0 0 0" rpy="0 0 0"/>
-            <inertia
-                     ixx="0.1"
-                     iyy="0.1"
-                     izz="0.1"
-                     ixy="0.0" ixz="0.0" iyz="0.0"
-            />
-        </inertial>
-        <visual>
-            <origin xyz="0 0 0" rpy="0 0 0"/>
-            <geometry>
-                <box size='0.03 0.03 0.1'/>
-            </geometry>
-        </visual>
-    </link>
-    <link name="front_right_strut">
-        <collision>
-            <origin xyz="0 0 0" rpy="0 0 0"/>
-            <geometry>
-                <box size='0.03 0.03 0.1'/>
-            </geometry>
-        </collision>
-        <inertial>
-            <mass value="0.2"/>
-            <origin xyz="0 0 0" rpy="0 0 0"/>
-            <inertia
-                     ixx="0.1"
-                     iyy="0.1"
-                     izz="0.1"
-                     ixy="0.0" ixz="0.0" iyz="0.0"
-                     />
-        </inertial>
-        <visual>
-            <origin xyz="0 0 0" rpy="0 0 0"/>
-            <geometry>
-                <box size='0.03 0.03 0.1'/>
-            </geometry>
-        </visual>
-    </link>
-    <gazebo reference="front_left_strut">
-        <material>Gazebo/DarkGrey</material>
-    </gazebo>
-    <gazebo reference="front_right_strut">
-        <material>Gazebo/DarkGrey</material>
-    </gazebo>
     <gazebo reference="front_left_wheel">
         <material>Gazebo/Black</material>
@@ -467,34 +412,18 @@
     </gazebo>
     <joint name="front_left_wheel_bearing" type="continuous">
-        <origin xyz="0 0.032 0" rpy="0 0 0"/>
+        <origin xyz="0.175 0.17 0" rpy="0 0 0"/>
         <child link="front_left_wheel"/>
-        <parent link="front_left_strut"/>
+        <parent link="chassis"/>
         <axis xyz="0 1 0" rpy="0 0 0"/>
-        <limit effort="10000" velocity="1000"/>
+        <limit effort="1000" velocity="1000"/>
         <dynamics damping="0.005" friction="0.005"/>
     </joint>
-    <joint name="front_left_steer_bearing" type="continuous">
-        <origin xyz='0.175 0.18 0' rpy="0 0 0"/>
-        <child link="front_left_strut"/>
+     <joint name="front_right_wheel_bearing" type="continuous">
+        <origin xyz="0.175 -0.17 0" rpy="0 0 0"/>
+        <child link="front_right_wheel"/>
         <parent link="chassis"/>
-        <axis xyz="0 0 1" rpy="0 0 0"/>
-        <limit effort="1000" velocity="1000"/>
-        <dynamics damping="0.1" friction="0.1"/>
-    </joint>
-     <joint name="front_right_wheel_bearing" type="continuous">
-        <origin xyz="0 -0.032 0" rpy="0 0 0"/>
-        <child link="front_right_wheel"/>
-        <parent link="front_right_strut"/>
         <axis xyz="0 1 0" rpy="0 0 0"/>
-        <limit effort="10000" velocity="1000"/>
+        <limit effort="1000" velocity="1000"/>
         <dynamics damping="0.005" friction="0.005"/>
-    </joint>
-    <joint name="front_right_steer_bearing" type="continuous">
-        <origin xyz='0.175 -0.18 0' rpy="0 0 0"/>
-        <child link="front_right_strut"/>
-        <parent link="chassis"/>
-        <axis xyz="0 0 1" rpy="0 0 0"/>
-        <limit effort="1000" velocity="1000"/>
-        <dynamics damping="0.1" friction="0.1"/>
     </joint>
     <!-- REAR WHEELS \\\\\\\\\\\\\\\\\\\\\\\\\\\\\\\\\\\\\\\\\\\\\\\\\-->
@@ -507,5 +436,5 @@
         </collision>
         <inertial>
-            <mass value="1.0"/>
+            <mass value="2.0"/>
             <origin xyz="0 0 0" rpy="0 1.5707 1.5707"/>
             <inertia
@@ -531,5 +460,5 @@
         </collision>
         <inertial>
-            <mass value="1.0"/>
+            <mass value="2.0"/>
             <origin xyz="0 0 0" rpy="0 1.5707 1.5707"/>
             <inertia
@@ -547,59 +476,4 @@
         </visual>
     </link>
-    <!-- Strut dims are derived from the dims of the wheel they carry -->
-    <link name="rear_left_strut">
-        <collision>
-            <origin xyz="0 0 0" rpy="0 0 0"/>
-            <geometry>
-                <box size='0.03 0.03 0.1'/>
-            </geometry>
-        </collision>
-        <inertial>
-            <mass value="0.2"/>
-            <origin xyz="0 0 0" rpy="0 0 0"/>
-            <inertia
-                     ixx="0.1"
-                     iyy="0.1"
-                     izz="0.1"
-                     ixy="0.0" ixz="0.0" iyz="0.0"
-                     />
-        </inertial>
-        <visual>
-            <origin xyz="0 0 0" rpy="0 0 0"/>
-            <geometry>
-                <box size='0.03 0.03 0.1'/>
-            </geometry>
-        </visual>
-    </link>
-    <link name="rear_right_strut">
-        <collision>
-            <origin xyz="0 0 0" rpy="0 0 0"/>
-            <geometry>
-                <box size='0.03 0.03 0.1'/>
-            </geometry>
-        </collision>
-        <inertial>
-            <mass value="2.0"/>
-            <origin xyz="0 0 0" rpy="0 0 0"/>
-            <inertia
-                     ixx="0.1"
-                     iyy="0.1"
-                     izz="0.1"
-                     ixy="0.0" ixz="0.0" iyz="0.0"
-                     />
-        </inertial>
-        <visual>
-            <origin xyz="0 0 0" rpy="0 0 0"/>
-            <geometry>
-                <box size='0.03 0.03 0.1'/>
-            </geometry>
-        </visual>
-    </link>
-    <gazebo reference="rear_left_strut">
-        <material>Gazebo/DarkGrey</material>
-    </gazebo>
-    <gazebo reference="rear_right_strut">
-        <material>Gazebo/DarkGrey</material>
-    </gazebo>
     <gazebo reference="rear_left_wheel">
         <material>Gazebo/Black</material>
@@ -609,34 +483,18 @@
     </gazebo>
     <joint name="rear_left_wheel_bearing" type="continuous">
-        <origin xyz="0 0.032 0" rpy="0 0 0"/>
+        <origin xyz="-0.175 0.17 0" rpy="0 0 0"/>
         <child link="rear_left_wheel"/>
-        <parent link="rear_left_strut"/>
+        <parent link="chassis"/>
         <axis xyz="0 1 0" rpy="0 0 0"/>
-        <limit effort="10000" velocity="1000"/>
+        <limit effort="1000" velocity="1000"/>
         <dynamics damping="0.005" friction="0.005"/>
     </joint>
-    <joint name="rear_left_steer_bearing" type="fixed">
-        <origin xyz='-0.175 0.18 0' rpy="0 0 0"/>
-        <child link="rear_left_strut"/>
+    <joint name="rear_right_wheel_bearing" type="continuous">
+        <origin xyz="-0.175 -0.17 0" rpy="0 0 0"/>
+        <child link="rear_right_wheel"/>
         <parent link="chassis"/>
-        <axis xyz="0 0 1" rpy="0 0 0"/>
-        <limit effort="1000" velocity="1000"/>
-        <dynamics damping="0.1" friction="0.1"/>
-    </joint>
-    <joint name="rear_right_wheel_bearing" type="continuous">
-        <origin xyz="0 -0.032 0" rpy="0 0 0"/>
-        <child link="rear_right_wheel"/>
-        <parent link="rear_right_strut"/>
         <axis xyz="0 1 0" rpy="0 0 0"/>
-        <limit effort="10000" velocity="1000"/>
+        <limit effort="1000" velocity="1000"/>
         <dynamics damping="0.005" friction="0.005"/>
     </joint>
-    <joint name="rear_right_steer_bearing" type="fixed">
-        <origin xyz='-0.175 -0.18 0' rpy="0 0 0"/>
-        <child link="rear_right_strut"/>
-        <parent link="chassis"/>
-        <axis xyz="0 0 1" rpy="0 0 0"/>
-        <limit effort="1000" velocity="1000"/>
-        <dynamics damping="0.1" friction="0.1"/>
-    </joint>
 </robot>

Commit message: chassis height fix

File: my_robot/urdf/sad_robot.xacro (robot description, xacro)
@@ -4,5 +4,5 @@
     <link name="robot_footprint"/>
     <joint name="robot_footprint_joint" type="fixed">
-        <origin xyz="0 0 0" rpy="0 0 0" />
+        <origin xyz="0 0 0.1" rpy="0 0 0" />
         <parent link="robot_footprint"/>
         <child link="chassis"/>
